File: KiCad_Nixie_Socket/GR_Nixie_Socket.sch (KiCad schematic (older format))
At the start: 5 parts, among them J1 Conn_01x06, J2 Conn_01x07

Commit message: Add files via upload
Connections:
- net Digit10 renamed Digit0
Changed lines of the file:
@@
 Digit9
 Text Label 1850 4400 0    50   ~ 0
-Digit10
+Digit0
 Text Label 1850 4500 0    50   ~ 0
 LeftDecimal
